File: helios/power.kicad_sch (KiCad schematic)
At the start: 7 parts, among them J1 Conn_01x03

Commit message: finish PCB + rename project
Parts:
- removed H1, H2, H3, H4: MountingHole, MountingHole:MountingHole_3.2mm_M3, symbol Mechanical:MountingHole
Other:
- moved on the sheet: C1, C2, J1
