File: helios/helios.kicad_pcb (KiCad board)
At the start: 2 copper layers, 150 x 105.9 mm, 64 parts, among them J1 Conn_01x03, J2 RELAY, Q1 BC557, Q2 BC557, Q3 BC557, Q4 BC557, Q5 BC557, Q6 BC557, Q7 BC557, Q8 BC557, SW1 RotaryEncoder, SW2 SW_Push, SW3 SW_Push, SW4 SW_Push, U1 74HC595, U2 74HC138, U3 CC56-12EWA, U4 74HC595, U5 74HC138, U6 CC56-12EWA

Commit message: finish PCB + rename project
Parts:
- added H10: MountingHole, MountingHole:MountingHole_3.2mm_M3, F.Cu at (166.4, 167.6)
- added H5: MountingHole, Relay_THT:Relay_Module_5V_Mounting, F.Cu at (144.8, 74.9)
- added H9: MountingHole, MountingHole:MountingHole_3.2mm_M3, F.Cu at (124.5, 167.6)
- J2: value RELAY -> Conn_01x04
- R1, R2, R3: value 10K -> 10k
- R10, R27, R28, R29, R30, R7, R8, R9: value 1K -> 1k
- SW1: value RotaryEncoder -> RotaryEncoder_Switch
- moved C1 104.4 mm to (168.9, 104.1), turned to 180 degrees
- moved C2 100.5 mm to (160.0, 104.1)
- moved J1 98.6 mm to (163.8, 99.0), turned to 90 degrees
- moved R4 66.6 mm to (134.0, 146.7), turned to 180 degrees
- moved R6 63.7 mm to (134.0, 153.0), turned to 180 degrees
- moved R5 58.8 mm to (134.0, 149.9), turned to 180 degrees
- moved SW2 57.3 mm to (120.1, 143.2), turned to 180 degrees
- moved C8 44.7 mm to (88.9, 147.3)
- moved SW4 38.7 mm to (93.4, 143.2), turned to 180 degrees
- moved C7 34.6 mm to (102.3, 147.3)
- moved SW3 28.6 mm to (106.8, 143.2), turned to 180 degrees
- moved C6 27.8 mm to (115.6, 147.3)
- moved J2 25.0 mm to (127.0, 109.2), turned to 0 degrees
- moved A1 16.5 mm to (137.2, 129.5)
Connections:
- A1 pad 4: GND -> unconnected-(A1-GND-Pad4)
Routing:
- net SPI_DATA_OUT: track 8.15 -> 349.2 mm
- net +3V3: track 379.8 -> 651.9 mm, vias 10 -> 13
- net ENABLE_ALARM: track 0.00 -> 182.2 mm, vias 0 -> 2
- net SPI_CLK: track 58.7 -> 233.7 mm, vias 2 -> 5
- net LATCH_ALARM: track 5.62 -> 166.8 mm, vias 1 -> 4
- net GND: track 223.6 -> 361.0 mm
- net SEL_A: track 58.2 -> 190.1 mm, vias 2 -> 4
- net SEL_B: track 51.4 -> 180.7 mm, vias 2 -> 4
- net SEL_C: track 45.2 -> 171.9 mm, vias 2 -> 4
- net RELAY_SIG: track 0.00 -> 100.9 mm, vias 0 -> 4
- net SPI_DATA: track 71.3 -> 150.9 mm, vias 1 -> 2
- net BTN_MANUAL: track 0.00 -> 77.9 mm, vias 0 -> 1
- net LATCH_TIME: track 58.3 -> 135.7 mm, vias 1 -> 2
- net ENC_SW: track 85.9 -> 158.2 mm, vias 1 -> 2
- net BTN_EDIT_ALARM: track 0.00 -> 64.3 mm, vias 0 -> 1
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Other:
- board size 150 x 105.9 mm -> 150 x 124.5 mm
- board text added: "<-"
- board text added: "ALARM"
- board text added: "RELAY 10A 250VAC"
- board text added: "TIME"

Commit message: small PCB fixes + print
Parts:
- J1: value Conn_01x03 -> To Relay
- J2: value Conn_01x04 -> DS3231
- R1, R2, R3, R4, R5, R6: value 10k -> 10K
- R10, R27, R28, R29, R30, R7, R8, R9: value 1k -> 1K
- SW1: value RotaryEncoder_Switch -> Rotary Encoder
- moved H1 14.1 mm to (75.5, 36.8)
- moved H2 14.1 mm to (217.7, 36.8)
- moved R5 12.8 mm to (135.8, 137.2)
- moved H5 12.8 mm to (146.6, 62.2)
- moved R1 12.8 mm to (167.5, 124.8)
- moved R10 12.8 mm to (208.8, 78.7)
- moved R17 12.8 mm to (201.2, 86.4)
- moved R19 12.8 mm to (95.8, 45.6)
- moved R20 12.8 mm to (103.4, 45.6)
- moved R21 12.8 mm to (103.4, 86.2)
- moved R22 12.8 mm to (95.8, 86.2)
- moved R23 12.8 mm to (92.0, 86.2)
- moved R24 12.8 mm to (99.6, 45.6)
- moved R25 12.8 mm to (107.2, 86.2)
- moved R26 12.8 mm to (99.6, 86.2)
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Routing:
- net SDA: track 50.2 -> 57.0 mm
- net GND: track 361.0 -> 364.2 mm
- net /Display_Time/DIG4: track 38.5 -> 40.8 mm
- net +3V3: track 651.9 -> 649.6 mm
- net /Display_Time/DIG3: track 37.1 -> 39.3 mm
- net /Display_Alarm/DIG8: track 39.5 -> 40.8 mm
- net ENABLE_ALARM: track 182.2 -> 183.3 mm
- net LATCH_ALARM: track 166.8 -> 167.8 mm
- net SPI_CLK: track 233.7 -> 234.7 mm
- net /Display_Alarm/DIG7: track 38.5 -> 39.3 mm
- net SCL: track 50.5 -> 50.0 mm
Other:
- board size 150 x 124.5 mm -> 149.9 x 125.7 mm
- board text added: "Arduino Nano"
- board text added: "EDIT ALARM"
- board text added: "EDIT TIME"
- board text added: "Helios Real-Time Lamp Controller https://github.com/kyriosaa/helios"
- board text added: "MANUAL"
- board text added: "Push"
