File: 2layer/helios/display_alarm.kicad_sch (KiCad schematic)
At the start: 19 parts, among them Q5 BC557, Q6 BC557, Q7 BC557, Q8 BC557, U4 74HC595, U5 74HC138, U6 CC56-12EWA

Commit message: added MCU code + documentation
Parts:
- R19, R20, R21, R22, R23, R24, R25, R26: value 150 -> 330
- U6: value CC56-12EWA -> CA56-12EWA
Connections:
- net +3V3 renamed +5V
