File: 2layer/helios/display_time.kicad_sch (KiCad schematic)
At the start: 19 parts, among them Q1 BC557, Q2 BC557, Q3 BC557, Q4 BC557, U1 74HC595, U2 74HC138, U3 CC56-12EWA

Commit message: added MCU code + documentation
Parts:
- R11, R12, R13, R14, R15, R16, R17, R18: value 150 -> 330
- U3: value CC56-12EWA -> CA56-12EWA
Connections:
- net +3V3 renamed +5V
