File: 2layer/helios/inputs.kicad_sch (KiCad schematic)
At the start: 16 parts, among them SW1 RotaryEncoder_Switch, SW2 SW_Push, SW3 SW_Push, SW4 SW_Push

Commit message: added MCU code + documentation
Connections:
- net +3V3 renamed +5V
