File: 2layer/helios/helios.kicad_pcb (KiCad board)
At the start: 2 copper layers, 149.9 x 125.7 mm, 67 parts, among them J1 To Relay, J2 DS3231, Q1 BC557, Q2 BC557, Q3 BC557, Q4 BC557, Q5 BC557, Q6 BC557, Q7 BC557, Q8 BC557, SW1 Rotary Encoder, SW2 SW_Push, SW3 SW_Push, SW4 SW_Push, U1 74HC595, U2 74HC138, U3 CC56-12EWA, U4 74HC595, U5 74HC138, U6 CC56-12EWA

Commit message: added MCU code + documentation
Parts:
- J1: value To Relay -> Conn_01x03
- J2: value DS3231 -> Conn_01x04
- R1, R2, R3, R4, R5, R6: value 10K -> 10k
- R10, R27, R28, R29, R30, R7, R8, R9: value 1K -> 1k
- R11, R12, R13, R14, R15, R16, R17, R18, R19, R20, R21, R22, R23, R24, R25, R26: value 150 -> 330
- SW1: value Rotary Encoder -> RotaryEncoder_Switch
Connections:
- A1 pad 17: +3V3 -> unconnected-(A1-3V3-Pad17)
- C2 pad 1: +3V3 -> +5V
- J2 pad 3: +3V3 -> +5V
- Q1 pad 3: +3V3 -> +5V
- Q2 pad 3: +3V3 -> +5V
- Q3 pad 3: +3V3 -> +5V
- Q4 pad 3: +3V3 -> +5V
- Q5 pad 3: +3V3 -> +5V
- Q6 pad 3: +3V3 -> +5V
- Q7 pad 3: +3V3 -> +5V
- Q8 pad 3: +3V3 -> +5V
- R1 pad 1: +3V3 -> +5V
- R2 pad 1: +3V3 -> +5V
- R3 pad 1: +3V3 -> +5V
- SW2 pad 2: +3V3 -> +5V
- SW3 pad 2: +3V3 -> +5V
- SW4 pad 2: +3V3 -> +5V
- U1 pad 10: +3V3 -> +5V
- U1 pad 16: +3V3 -> +5V
- U2 pad 16: +3V3 -> +5V
- U2 pad 6: +3V3 -> +5V
- U4 pad 10: +3V3 -> +5V
- U4 pad 16: +3V3 -> +5V
- U5 pad 16: +3V3 -> +5V
- U5 pad 6: +3V3 -> +5V
Routing:
- net +5V: track 57.2 -> 709.4 mm, vias 2 -> 15
- net +3V3: track 649.6 -> 0.00 mm, vias 13 -> 0
- net GND: track 364.2 -> 420.6 mm, vias 0 -> 2

Commit message: PCB CC->CA footprint fix + display blink rate adjustment
Parts:
- U3, U6: value CC56-12EWA -> CA56-12EWA
