File: 4layer/helios/helios.kicad_pcb (KiCad board)
At the start: 4 copper layers, 149.9 x 125.7 mm, 67 parts, among them J1 To Relay, J2 DS3231, Q1 BC557, Q2 BC557, Q3 BC557, Q4 BC557, Q5 BC557, Q6 BC557, Q7 BC557, Q8 BC557, SW1 RotaryEncoder, SW2 SW_Push, SW3 SW_Push, SW4 SW_Push, U1 74HC595, U2 74HC138, U3 CC56-12EWA, U4 74HC595, U5 74HC138, U6 CC56-12EWA

Commit message: update 4layer board
Parts:
- removed ?: , 
- added G***: LOGO, LOGO, F.Cu at (147.0, 99.0)
- moved R25 0.14 mm to (107.2, 86.4)
- moved R21 0.14 mm to (103.4, 86.4)
- moved R22 0.14 mm to (95.8, 86.4)
- moved R23 0.14 mm to (92.0, 86.4)
- moved R26 0.14 mm to (99.6, 86.4)
Routing:
- net SPI_CLK: track 76.6 -> 206.6 mm
- net ENC_SW: track 9.57 -> 122.2 mm, vias 0 -> 2
- net SPI_DATA: track 0.00 -> 101.0 mm
- net LATCH_TIME: track 0.00 -> 89.3 mm
- net SPI_DATA_OUT: track 0.00 -> 85.3 mm, vias 0 -> 2
- net RELAY_SIG: track 0.00 -> 82.9 mm
- net ENC_DT: track 10.0 -> 71.0 mm, vias 0 -> 1
- net ENC_CLK: track 10.0 -> 69.8 mm, vias 0 -> 1
- net SDA: track 0.00 -> 53.5 mm, vias 0 -> 1
- net SCL: track 0.00 -> 50.7 mm, vias 0 -> 1
- net +5V: track 6.89 -> 51.9 mm, vias 0 -> 3
Other:
- outline, holes or cut-outs redrawn
- board text added: "10A 250VAC"
- board text removed: "NANO"
- board text removed: "RELAY 10A 250VAC"

Commit message: more pixel assets for the 4layer board
Parts:
- added G***: LOGO, LOGO, F.Cu at (185.0, 91.8)
- added G***: LOGO, LOGO, F.Cu at (83.0, 37.8)
- added G***: LOGO, LOGO, F.Cu at (101.4, 128.3)
- added G***: LOGO, LOGO, F.Cu at (165.0, 54.2)
- added G***: LOGO, LOGO, F.Cu at (202.2, 100.2)
- added G***: LOGO, LOGO, F.Cu at (216.2, 45.8)
- added G***: LOGO, LOGO, F.Cu at (180.0, 36.5)
- added G***: LOGO, LOGO, F.Cu at (99.5, 95.8)
- added G***: LOGO, LOGO, F.Cu at (114.7, 128.3)
- added G***: LOGO, LOGO, F.Cu at (108.2, 100.2)
- added G***: LOGO, LOGO, F.Cu at (100.2, 119.5)
- added G***: LOGO, LOGO, F.Cu at (193.5, 95.8)
- added G***: LOGO, LOGO, F.Cu at (115.8, 36.2)
- added G***: LOGO, LOGO, F.Cu at (76.8, 48.8)
- added G***: LOGO, LOGO, F.Cu at (123.0, 43.8)
- added G***: LOGO, LOGO, F.Cu at (207.0, 37.8)
- added G***: LOGO, LOGO, F.Cu at (81.8, 42.2)
- added G***: LOGO, LOGO, F.Cu at (127.8, 53.0)
- added G***: LOGO, LOGO, F.Cu at (88.0, 128.3)
- added G***: LOGO, LOGO, F.Cu at (170.0, 42.8)
- added G***: LOGO, LOGO, F.Cu at (91.0, 91.8)
- SW1: value RotaryEncoder -> Rotary Encoder
- moved C6 4.00 mm to (113.4, 134.6)
- moved C7 4.00 mm to (100.2, 134.6)
- moved C8 4.00 mm to (86.7, 134.6)
- moved SW2 4.00 mm to (117.9, 130.5)
- moved SW3 4.00 mm to (104.7, 130.5)
- moved SW4 4.00 mm to (91.2, 130.5)
- moved U1 0.73 mm to (213.4, 104.1)
- moved U2 0.73 mm to (174.0, 111.8)
- moved U4 0.71 mm to (119.4, 104.2)
- moved U5 0.71 mm to (80.0, 111.9)
Routing:
- net BTN_EDIT_ALARM: track 51.1 -> 56.2 mm
- net BTN_EDIT_TIME: track 28.4 -> 32.4 mm
- net BTN_MANUAL: track 66.3 -> 68.8 mm
- net /Display_Time/DIG3: track 38.6 -> 36.4 mm
- net /Display_Alarm/DIG7: track 38.6 -> 36.5 mm
- net /Display_Time/DIG4: track 39.0 -> 37.1 mm
- net /Display_Alarm/DIG8: track 39.0 -> 37.2 mm
- net /Display_Time/DIG1: track 19.1 -> 18.2 mm
- net SPI_CLK: track 206.6 -> 205.7 mm
- net /Display_Alarm/DIG5: track 19.1 -> 18.3 mm
- net /Display_Alarm/SEG_F: track 99.8 -> 99.0 mm
- net ENABLE_TIME: track 50.1 -> 50.9 mm
- net /Display_Time/SEG_F: track 99.8 -> 99.0 mm
- net /Display_Time/SEG_E: track 31.5 -> 32.2 mm
- net /Display_Time/SEG_A: track 103.7 -> 103.0 mm
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Other:
- board text added: "x"
